File: pcbs/tonyverse.kicad_pcb (KiCad board)
At the start: 2 copper layers, 259.2 x 108.6 mm, 62 parts

Commit message: egg
Routing:
- net P2: track 107.7 -> 141.5 mm
- net P4: track 196.0 -> 219.1 mm
- net P6: track 312.3 -> 333.9 mm
- net P5: track 272.0 -> 287.9 mm
- net P20: track 126.7 -> 140.6 mm
- net P21: track 130.7 -> 144.6 mm
- net P0: track 119.3 -> 133.2 mm
- net P1: track 119.6 -> 133.5 mm
- net P7: track 392.1 -> 400.3 mm
- net P9: track 67.4 -> 74.4 mm
- net P10: track 70.0 -> 77.0 mm
- net P3: track 163.5 -> 170.1 mm
- net mirror_pinky_top: track 11.3 -> 15.1 mm
- net index_top: track 12.3 -> 15.4 mm
- net mirror_better_top: track 12.0 -> 15.1 mm
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